Commit message: Encoder based drive odometry

File: mirv_description/urdf/cameras/rgbd/orbbec_astra.urdf.xacro (robot description, xacro)
@@ -107,5 +107,5 @@
                          <clip>
                               <near>0.05</near>
-                              <far>35</far>
+                              <far>3.5</far>
                          </clip>
                     </camera>

File: mirv_description/urdf/dd_controller.urdf.xacro (robot description, xacro)
@@ -11,9 +11,9 @@
         <odometryTopic>odom</odometryTopic>
         <odometryFrame>odom</odometryFrame>
-        <odometrySource>world</odometrySource>
-        <publishOdomTF>true</publishOdomTF>
+<!--        <odometrySource>world</odometrySource>-->
+<!--        <publishOdomTF>true</publishOdomTF>-->
         <robotBaseFrame>base_footprint</robotBaseFrame>
-<!--        <publishWheelTF>false</publishWheelTF>-->
-        <publishTf>true</publishTf>
+        <publishWheelTF>false</publishWheelTF>
+<!--        <publishTf>true</publishTf>-->
 <!--        <publishWheelJointState>true</publishWheelJointState>-->
 <!--        <legacyMode>false</legacyMode>-->

File: mirv_description/urdf/lidars/vlp_16.urdf.xacro (robot description, xacro)
@@ -1,5 +1,4 @@
 <?xml version="1.0"?>
-<robot name="sensor_vlp_16" xmlns:xacro="http://ros.org/wiki/xacro">
-	<xacro:include filename="$(find mirv_description)/urdf/includes/materials.urdf.xacro"/>
+<robot xmlns:xacro="http://ros.org/wiki/xacro" name="VLP-16">
   <xacro:property name="M_PI" value="3.1415926535897931" />
   <xacro:macro name="sensor_vlp_16" params="*origin visualize:=false parent:=base_link name:=velodyne topic:=/velodyne_points hz:=10 lasers:=16 samples:=1875 collision_range:=0.3 min_range:=0.9 max_range:=130.0 noise:=0.008 min_angle:=-${M_PI} max_angle:=${M_PI} color:=black">
@@ -7,7 +6,7 @@
       <xacro:insert_block name="origin" />
       <parent link="${parent}"/>
-      <child link="${name}_link"/>
+      <child link="${name}_base_link"/>
     </joint>
-    <link name="${name}_link">
+    <link name="${name}_base_link">
       <inertial>
         <mass value="0.83"/>
@@ -34,7 +33,7 @@
       </collision>
     </link>
-    <joint name="${name}_joint" type="fixed" >
+    <joint name="${name}_base_scan_joint" type="fixed" >
       <origin xyz="0 0 0.0377" rpy="0 0 0" />
-      <parent link="${name}_link" />
+      <parent link="${name}_base_link" />
       <child link="${name}"/>
     </joint>
@@ -54,5 +53,5 @@
     <!-- Gazebo requires the velodyne_gazebo_plugins package -->
     <gazebo reference="${name}">
-      <sensor type="ray" name="${name}-VLP16">
+      <sensor type="gpu_ray" name="${name}-VLP16">
         <pose>0 0 0 0 0 0</pose>
         <visualize>${visualize}</visualize>
@@ -81,14 +80,10 @@
             <type>gaussian</type>
             <mean>0.0</mean>
-            <stddev>0.01</stddev>
+            <stddev>0.0</stddev>
           </noise>
         </ray>
-        <plugin name="${name}_controller" filename="libgazebo_ros_velodyne_laser.so">
+        <plugin name="gazebo_ros_laser_controller" filename="libgazebo_ros_gpu_laser.so">
           <topicName>${topic}/points</topicName>
           <frameName>${name}</frameName>
-          <organize_cloud>false</organize_cloud>
-          <min_range>${min_range}</min_range>
-          <max_range>${max_range}</max_range>
-          <gaussianNoise>${noise}</gaussianNoise>
         </plugin>
       </sensor>

File: mirv_description/urdf/mirv_gazebo.urdf.xacro (robot description, xacro)
@@ -44,17 +44,17 @@
   <xacro:arg name="robot_name" default="mirv" />
   <xacro:property name="robot_name_prop" value="$(arg robot_name)" />
- <!-- <gazebo>
-   Publish current joint angles
-   <plugin name="joint_state_publisher" filename="libgazebo_ros_joint_state_publisher.so">
-       <xacro:if value="${robot_name_prop != ''}" >
-         <robotNamespace>$(arg robot_name)</robotNamespace>
-       </xacro:if>
-       <jointName>
-           wheel_fl, wheel_fr, wheel_rl, wheel_rr
-       </jointName>
-       <updateRate>100</updateRate>
-       <alwaysOn>true</alwaysOn>
-   </plugin>
- </gazebo> -->
+<!--  <gazebo>-->
+<!--    &lt;!&ndash; Publish current joint angles &ndash;&gt;-->
+<!--    <plugin name="joint_state_publisher" filename="libgazebo_ros_joint_state_publisher.so">-->
+<!--        <xacro:if value="${robot_name_prop != ''}" >-->
+<!--          <robotNamespace>$(arg robot_name)</robotNamespace>-->
+<!--        </xacro:if>-->
+<!--        <jointName>-->
+<!--            wheel_fl, wheel_fr, wheel_rl, wheel_rr-->
+<!--        </jointName>-->
+<!--        <updateRate>100</updateRate>-->
+<!--        <alwaysOn>true</alwaysOn>-->
+<!--    </plugin>-->
+<!--  </gazebo>-->
   <link name="base_footprint"/>
   <link name="base_link">
@@ -112,23 +112,14 @@
   <!-- Vehicle controller -->
   <xacro:dd_controller name="mirv_controller" wheelbase="${2*half_wheelbase}" wheel_diameter="${2*wheel_radius}" left_joint="wheel_fl_joint" right_joint="wheel_fr_joint" />
-  <!-- LiDAR Velodyne VLP-16 -->
-  <!-- 16-beam lidar, +- 15 deg vertical and 360 deg horizontal FoV at 10hz -->
-  <xacro:sensor_vlp_16 name="lidar" parent="base_link" color="black" visualize="true">
+  <!-- LiDAR Hokuyo ust10lx -->
+  <xacro:sensor_hokuyo_ust10lx name="lidar" parent="base_link" color="black" visualize="true">
     <origin xyz="0.25 0 0.4" rpy="0 0 0"/>
-  </xacro:sensor_vlp_16>
-  <!-- LiDAR Hokuyo ust10lx -->
-  <!-- <xacro:sensor_hokuyo_ust10lx name="lidar" parent="base_link" color="black" visualize="true">
-    <origin xyz="0.25 0 0.4" rpy="0 0 0"/>
-  </xacro:sensor_hokuyo_ust10lx> -->
-  <!-- Wheel encoders -->
-  <!-- <xacro:macro name="sensor_rotary_encoder" params="ns:=/ parent joint:=front_left_wheel_rev d:=0.15 topic:=/encoder update_rate:=100.0 ppr:=150"> -->
-<!--  <xacro:sensor_rotary_encoder ns="/" parent="wheel_fl" joint="wheel_fl_joint" d="${wheel_radius}" topic="/wheel_fl_encoder" update_rate="100.0" ppr="150"/>-->
+  </xacro:sensor_hokuyo_ust10lx>
+<!--  <xacro:sensor_hokuyo_ust10lx_gazebo name="lidar"/>-->
   <!-- Camera Orbbec Astra -->
-  <!-- RGBD binocular camera, 640x480p 20fps -->
   <xacro:sensor_orbbec_astra name="camera" parent="base_link" color="blue">
     <origin xyz="0 0 0.5" rpy="0 0 0" />
   </xacro:sensor_orbbec_astra>
   <!-- IMU -->
-  <!-- IMU with params described below. No real through put into it yet. -->
   <xacro:sensor_modified_imu name="imu" parent="base_link" color="red"
                   update_rate="10.0"
@@ -146,5 +137,4 @@
   </xacro:sensor_modified_imu>
   <!-- GPS w/ Variable Dropouts-->
-  <!-- GPS starting at the reference position with noise/params described below -->
   <xacro:sensor_standard_gps name="gps" parent="base_link" color="white"
                   ref_lat="40.1021496545"
@@ -158,4 +148,5 @@
     <origin xyz="-0.14 0 0.12" rpy="0 0 0"/>
   </xacro:sensor_standard_gps>
+<!--  <xacro:sensor_standard_gps_gazebo name="gps" ref_lat="1" ref_long="2" ref_head="3" drift="4" vel_drift="5" noise="6" vel_noise="7" update_rate="8"/>-->
   <!-- Simple Simulated Battery -->
   <!-- <xacro:sensor_battery_approx/>-->
