Commit message: Got the simulation into a working state, GPS and IMU now read good values

File: mirv_description/urdf/gps/gps_standard.urdf.xacro (robot description, xacro)
@@ -2,5 +2,5 @@
 <robot name="sensor_standard_gps" xmlns:xacro="http://ros.org/wiki/xacro">
 	<xacro:include filename="$(find mirv_description)/urdf/includes/materials.urdf.xacro"/>
-  	<xacro:macro name="sensor_standard_gps" params="name parent *origin color ref_lat ref_long ref_head drift vel_drift noise vel_noise update_rate">
+  	<xacro:macro name="sensor_standard_gps" params="name parent *origin color frame_id topic_name velocity_topic_name ref_lat ref_long ref_head drift vel_drift noise vel_noise update_rate">
 		<joint name="${name}_joint" type="fixed">
 			<axis xyz="0 1 0"/>
@@ -38,7 +38,7 @@
 				<updateRate>${update_rate}</updateRate>
 				<bodyName>${name}_link</bodyName>
-				<frameId>${name}_link</frameId>
-				<topicName>/fix</topicName>
-			  	<velocityTopicName>vel</velocityTopicName>
+				<frameId>${frame_id}</frameId>
+				<topicName>${topic_name}</topicName>
+			  	<velocityTopicName>${velocity_topic_name}</velocityTopicName>
 				<referenceLatitude>${ref_lat}</referenceLatitude>
 				<referenceLongitude>${ref_long}</referenceLongitude>

File: mirv_description/urdf/mirv_gazebo.urdf.xacro (robot description, xacro)
@@ -113,7 +113,7 @@
   <xacro:dd_controller name="mirv_controller" wheelbase="${2*half_wheelbase}" wheel_diameter="${2*wheel_radius}" left_joint="wheel_fl_joint" right_joint="wheel_fr_joint" />
   <!-- LiDAR Hokuyo ust10lx -->
-  <xacro:sensor_hokuyo_ust10lx name="lidar" parent="base_link" color="black" visualize="true">
-    <origin xyz="0.25 0 0.4" rpy="0 0 0"/>
-  </xacro:sensor_hokuyo_ust10lx>
+<!--  <xacro:sensor_hokuyo_ust10lx name="lidar" parent="base_link" color="black" visualize="true">-->
+<!--    <origin xyz="0.25 0 0.4" rpy="0 0 0"/>-->
+<!--  </xacro:sensor_hokuyo_ust10lx>-->
 <!--  <xacro:sensor_hokuyo_ust10lx_gazebo name="lidar"/>-->
   <!-- Camera Orbbec Astra -->
@@ -138,12 +138,15 @@
   <!-- GPS w/ Variable Dropouts-->
   <xacro:sensor_standard_gps name="gps" parent="base_link" color="white"
+				  frame_id="map"
+				  topic_name="/gps/fix"
+				  velocity_topic_name="/gps/vel"
                   ref_lat="40.1021496545"
                   ref_long="-88.2267974168"
-                  ref_head="90.0"
+                  ref_head="50.0"
                   update_rate="10.0"
                   drift="0.0"
-                  noise="0.001"
-                  vel_drift="0.00001"
-                  vel_noise="0.00001">
+                  noise="0.5"
+                  vel_drift="0.00"
+                  vel_noise="0.1">
     <origin xyz="-0.14 0 0.12" rpy="0 0 0"/>
   </xacro:sensor_standard_gps>

File: mirv_description/urdf/motion/imu_mod.urdf.xacro (robot description, xacro)
@@ -36,5 +36,5 @@
                <plugin name="${name}_controller" filename="libhector_gazebo_ros_imu.so">
                     <alwaysOn>true</alwaysOn>
-                    <topicName>/${name}</topicName>
+                    <topicName>/${name}_raw</topicName>
                     <topicNameCustom>/${name}/custom</topicNameCustom>
                     <serviceName>${name}/service</serviceName>
