Commit message: fixed python library issues, and got simulation working as far as I can tell

File: mirv_description/urdf/mirv_gazebo.urdf.xacro (robot description, xacro)
@@ -33,6 +33,6 @@
      ========================================================= -->
   <xacro:property name="half_track_width" value="0.25" />
-  <xacro:property name="half_wheelbase" value="0.15" />
-  <xacro:property name="wheel_radius" value="0.1" />
+  <xacro:property name="half_wheelbase" value="0.2179" />
+  <xacro:property name="wheel_radius" value="0.09229" />
   <xacro:property name="wheel_thickness" value="0.0508" />
   <xacro:property name="wheel_mass" value="0.5" />
